File: OctoBreakout.kicad_pcb (KiCad board)
At the start: 2 copper layers, 102.9 x 48.3 mm, 56 parts, among them J1 Screw_Terminal_1x02, J10 JC, J11 JD, J12 JE, J13 JF, J14 JG, J15 JH, J16 JA, J17 JB, J18 JC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

Commit message: monir revisions
Parts:
- added REF**: Drill_Hole, 1dah:Drill_Hole_0.125in, F.Cu at (175.8, 35.6)
- added REF**: Drill_Hole, 1dah:Drill_Hole_0.2in, F.Cu at (142.2, 36.3)
- added REF**: Drill_Hole, 1dah:Drill_Hole_0.2in, F.Cu at (167.6, 36.3)
- added REF**: Drill_Hole, 1dah:Drill_Hole_0.125in, F.Cu at (174.8, 91.7)
- added REF**: Drill_Hole, 1dah:Drill_Hole_0.125in, F.Cu at (79.8, 35.6)
- added REF**: Drill_Hole, 1dah:Drill_Hole_0.125in, F.Cu at (79.5, 90.9)
- added REF**: Drill_Hole, 1dah:Drill_Hole_0.2in, F.Cu at (91.4, 90.7)
- added REF**: Drill_Hole, 1dah:Drill_Hole_0.2in, F.Cu at (116.8, 90.7)
- added REF**: Drill_Hole, 1dah:Drill_Hole_0.2in, F.Cu at (142.2, 90.7)
- added REF**: Drill_Hole, 1dah:Drill_Hole_0.2in, F.Cu at (167.6, 90.7)
- added REF**: Drill_Hole, 1dah:Drill_Hole_0.2in, F.Cu at (91.4, 36.3)
- added REF**: Drill_Hole, 1dah:Drill_Hole_0.2in, F.Cu at (116.8, 36.3)
Routing:
- net /5V: track 82.4 -> 84.1 mm
Other:
- board size 102.9 x 48.3 mm -> 102.9 x 62 mm
- board text added: "+Data-"
- board text added: "Clk"
- board text added: "Data"
- board text removed: "+ D -"
